File: Hardware/eCAD/WEST_nrf52840_hydrophone_node/WEST_nrf52840_hydrophone_node.kicad_pcb (KiCad board)
At the start: 2 copper layers, 48.4 x 145.3 mm, 37 parts, among them J1 On/Off, J10 Conn_01x02_Pin, J2 RTC_Batt, J3 Uart1, J5 Mounting Hole, J6 Mounting Hole, J7 Mounting Hole, J8 Mounting Hole, Q1 2N7002, Q2 2N7002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

Commit message: Expand readme
Parts:
- moved U4 0.24 mm to (150.3, 25.2)
Routing:
- net GND: vias 35 -> 43
- net (no net): vias 1 -> 0
Other:
- outline, holes or cut-outs redrawn
Changed lines of the file:
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@@
 	(footprint "Project_Footprint_Lib:XIAO-nRF52840-DIP"
 		(layer "F.Cu")
-		(at 150.5685 25.25 90)
+		(at 150.33 25.25 90)
 		(property "Reference" "U4"
 			(at -8 -12 90)
@@
 		(attr smd)
 		(fp_line
-			(start -3.991272 -12.051)
-			(end 4.004 -12.051)
-			(stroke
-				(width 0.127)
-				(type solid)
-			)
-			(layer "F.SilkS")
-		)
-		(fp_line
-			(start 4.504 -11.551)
-			(end 4.504 -10.541)
-			(stroke
-				(width 0.127)
-				(type solid)
-			)
-			(layer "F.SilkS")
-		)
-		(fp_line
 			(start 6.985 -10.541)
 			(end -6.985 -10.541)
@@
 		)
 		(fp_line
-			(start -4.495 -10.541)
-			(end -4.491272 -11.551272)
+			(start -3.995272 -10)
+			(end 4 -10)
 			(stroke
 				(width 0.127)
@@
 		)
 		(fp_arc
-			(start 4.004 -12.051)
-			(mid 4.357524 -11.904524)
-			(end 4.504 -11.551)
-			(stroke
-				(width 0.127)
-				(type default)
-			)
-			(layer "F.SilkS")
-		)
-		(fp_arc
-			(start -4.491272 -11.551272)
-			(mid -4.344728 -11.90464)
-			(end -3.991272 -12.051)
-			(stroke
-				(width 0.127)
-				(type default)
-			)
-			(layer "F.SilkS")
-		)
-		(fp_arc
 			(start 6.985 -10.541)
 			(mid 8.332038 -9.983038)
@@
 	(gr_line
 		(start 159 13.5)
-		(end 142 13.5)
+		(end 141.414214 13.5)
 		(stroke
 			(width 0.0381)
@@
 	)
 	(gr_arc
-		(start 140 15.5)
-		(mid 140.585786 14.085786)
-		(end 142 13.5)
+		(start 139.414214 15.5)
+		(mid 140 14.085786)
+		(end 141.414214 13.5)
 		(stroke
 			(width 0.0381)
@@
 	)
 	(gr_line
-		(start 161 45.500006)
-		(end 161 15.5)
+		(start 117.5 35.552944)
+		(end 137.414214 35.552944)
 		(stroke
 			(width 0.0381)
@@
 	)
 	(gr_line
-		(start 138 35.552944)
-		(end 117.5 35.552944)
+		(start 161 45.500006)
+		(end 161 15.5)
 		(stroke
 			(width 0.0381)
@@
 	)
 	(gr_line
-		(start 140 15.5)
-		(end 140 33.552944)
+		(start 139.414214 15.5)
+		(end 139.414214 33.552944)
 		(stroke
 			(width 0.0381)
@@
 	)
 	(gr_arc
-		(start 140 33.552944)
-		(mid 139.414214 34.967158)
-		(end 138 35.552944)
+		(start 139.414214 33.552944)
+		(mid 138.828428 34.967158)
+		(end 137.414214 35.552944)
 		(stroke
 			(width 0.0381)
@@
 		)
 	)
-	(via
-		(at 195.6 80.5)
-		(size 0.6)
-		(drill 0.3)
-		(layers "F.Cu" "B.Cu")
-		(net 0)
-	)
 	(segment
 		(start 159.9 32.0415)
@@
 	)
 	(via
+		(at 152.25 49.25)
+		(size 0.6)
+		(drill 0.3)
+		(layers "F.Cu" "B.Cu")
+		(free yes)
+		(net 1)
+	)
+	(via
+		(at 160 78.25)
+		(size 0.6)
+		(drill 0.3)
+		(layers "F.Cu" "B.Cu")
+		(free yes)
+		(net 1)
+	)
+	(via
 		(at 125.8 136.1)
 		(size 0.6)
@@
 	)
 	(via
+		(at 136 36.75)
+		(size 0.6)
+		(drill 0.3)
+		(layers "F.Cu" "B.Cu")
+		(free yes)
+		(net 1)
+	)
+	(via
 		(at 153.15 99.4)
 		(size 0.6)
@@
 	)
 	(via
+		(at 159 79)
+		(size 0.6)
+		(drill 0.3)
+		(layers "F.Cu" "B.Cu")
+		(free yes)
+		(net 1)
+	)
+	(via
 		(at 136.25 74.65)
 		(size 0.6)
@@
 	)
 	(via
+		(at 148.75 46)
+		(size 0.6)
+		(drill 0.3)
+		(layers "F.Cu" "B.Cu")
+		(free yes)
+		(net 1)
+	)
+	(via
 		(at 137.6 74.6)
 		(size 0.6)
@@
 	)
 	(via
+		(at 136 37.75)
+		(size 0.6)
+		(drill 0.3)
+		(layers "F.Cu" "B.Cu")
+		(free yes)
+		(net 1)
+	)
+	(via
 		(at 136.5 46.65)
 		(size 0.6)
@@
 	)
 	(via
+		(at 136.75 36.75)
+		(size 0.6)
+		(drill 0.3)
+		(layers "F.Cu" "B.Cu")
+		(free yes)
+		(net 1)
+	)
+	(via
 		(at 129.3 128.6)
 		(size 0.6)
@@
 	)
 	(via
+		(at 159.9 38.5)
+		(size 0.6)
+		(drill 0.3)
+		(layers "F.Cu" "B.Cu")
+		(net 1)
+	)
+	(via
 		(at 114.6 147.35)
 		(size 0.6)
@@
 	)
 	(segment
-		(start 157.073 33.332056)
-		(end 157.073 18.7455)
-		(width 0.305)
-		(layer "B.Cu")
-		(net 39)
-	)
-	(segment
 		(start 143.75 88.17)
 		(end 143.9525 87.9675)
@@
 	)
 	(segment
-		(start 143.9525 46.452556)
-		(end 157.073 33.332056)
+		(start 156.75 33.655056)
+		(end 156.75 19.0685)
 		(width 0.305)
 		(layer "B.Cu")
@@
 	)
 	(segment
-		(start 157.073 18.7455)
+		(start 156.75 19.0685)
 		(end 158.1885 17.63)
 		(width 0.305)
@@
 		(width 0.305)
 		(layer "B.Cu")
+		(net 39)
+	)
+	(segment
+		(start 143.9525 46.452556)
+		(end 156.75 33.655056)
+		(width 0.305)
+		(layer "B.Cu")
